File: schemes/simple/weather station - simple - mirror.brd (EAGLE design)
At the start: 134.6 x 100 mm, 15 parts, among them IC1 7805TV, Q1 BC546B

Commit message: PCB scheme update
Parts:
- moved JP1 114.3 mm to (10.2, 24.1), flipped to the bottom
- moved JP2 114.3 mm to (10.2, 38.1), flipped to the bottom
- moved U$3 94.0 mm to (20.3, 69.8), flipped to the bottom
- moved U$4 81.3 mm to (108.0, 14.0), flipped to the bottom
- moved R3 76.2 mm to (105.4, 40.6), flipped to the bottom
- moved R1 66.0 mm to (34.3, 47.0), flipped to the bottom
- moved U$2 55.9 mm to (39.4, 36.8), flipped to the bottom
- moved R4 48.3 mm to (91.4, 40.6), flipped to the bottom
- moved Q1 40.6 mm to (47.0, 45.7), flipped to the bottom
- moved U$5 35.6 mm to (85.1, 48.3), flipped to the bottom
- moved U$1 30.5 mm to (52.1, 78.7), flipped to the bottom
- moved R2 20.3 mm to (77.5, 50.8), flipped to the bottom
- moved C2 15.2 mm to (59.7, 49.5), flipped to the bottom
- moved C1 2.54 mm to (68.6, 47.0), flipped to the bottom
- moved IC1 2.54 mm to (66.0, 48.3), flipped to the bottom
Routing:
- added copper zone on layer 1, net GND
- removed copper zone on layer 16, net GND
